File: KiCad_ASCEO/ASCEO.kicad_pcb (KiCad board)
At the start: 2 copper layers, 75 x 75 mm, 38 parts, among them J1 USB_OTG, J2 JST-XH 6-Pin (Motor + Encoder), J3 JST-XH 5-Pin (Raspberry Pi), J4 Barrel_Jack, J5 Screw_Terminal, SW1 RESET1, SW2 BOOT1, U1 ESP32-S3-WROOM-1-N4, U2 LDI1117-3.3H, U3 BMI323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

Commit message: Gerber and Drilling Files
Parts:
- moved D7 0.80 mm to (126.4, 119.3)
- renumbered SW2 to BOOT, SW1 to RESET
Routing:
- net +3V3: track 215.4 -> 214.4 mm
Changed lines of the file:
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@@
 			(plot_on_all_layers_selection 0x00000000_00000000_00000000_00000000)
 			(disableapertmacros no)
-			(usegerberextensions no)
+			(usegerberextensions yes)
 			(usegerberattributes yes)
 			(usegerberadvancedattributes yes)
@@
 			(outputformat 1)
 			(mirror no)
-			(drillshape 1)
+			(drillshape 0)
 			(scaleselection 1)
-			(outputdirectory "")
+			(outputdirectory "../Manufacturing/")
 		)
 	)
@@
 	(footprint "LED_SMD:LED_0805_2012Metric_Pad1.15x1.40mm_HandSolder"
 		(layer "F.Cu")
-		(at 127.224999 119.3443 180)
+		(at 126.424999 119.3443 180)
 		(descr "LED SMD 0805 (2012 Metric), square (rectangular) end terminal, IPC-7351 nominal, (Body size source: https://docs.google.com/spreadsheets/d/1BsfQQcO9C6DZCsRaXUlFlo91Tg2WpOkGARC1WS5S8t0/edit?usp=sharing), generated with kicad-footprint-generator")
 		(tags "LED handsolder")
 		(property "Reference" "D7"
-			(at 0 -1.65 0)
+			(at -0.225 1.7 0)
 			(layer "F.SilkS")
 			(effects
@@
 		)
 		(property "Value" "LED"
-			(at 0 1.65 0)
+			(at -0.025 1.7 0)
 			(layer "F.Fab")
 			(effects
@@
 			(effects
 				(font
-					(size 0.787402 0.787402)
+					(size 0.8 0.8)
 					(thickness 0.15)
 				)
@@
 			(effects
 				(font
-					(size 0.787402 0.787402)
+					(size 0.8 0.8)
 					(thickness 0.15)
 				)
@@
 		(layer "F.Cu")
 		(at 124.749999 82.8443 90)
-		(property "Reference" "SW1"
-			(at -0.325 -3.385 90)
+		(property "Reference" "RESET"
+			(at -0.2 -3.4 90)
 			(layer "F.SilkS")
 			(effects
@@
 		(fp_text user "*"
 			(at -2.032 -1 0)
-			(layer "F.SilkS")
-			(effects
-				(font
-					(size 1 1)
-					(thickness 0.15)
-				)
-			)
-		)
-		(fp_text user "*"
-			(at -2.032 -1 0)
 			(unlocked yes)
 			(layer "F.SilkS")
@@
 		(tags "capacitor handsolder")
 		(property "Reference" "C11"
-			(at -2.9375 0.04 0)
+			(at -3.1375 0.04 0)
 			(layer "F.SilkS")
 			(effects
@@
 		)
 		(fp_text user "*"
-			(at -1.61925 -2.6518 0)
-			(layer "F.SilkS")
-			(effects
-				(font
-					(size 1 1)
-					(thickness 0.15)
-				)
-			)
-		)
-		(fp_text user "*"
 			(at -0.4953 -1.4478 0)
 			(layer "F.Fab")
@@
 		(tags "capacitor handsolder")
 		(property "Reference" "C1"
-			(at 0 -1 0)
+			(at -1.0625 1.4 0)
 			(layer "F.SilkS")
 			(effects
@@
 		(layer "F.Cu")
 		(at 166.749999 86.3443 180)
-		(property "Reference" "SW2"
-			(at -0.325 -3.385 0)
+		(property "Reference" "BOOT"
+			(at 0.2 -3.5 0)
 			(layer "F.SilkS")
 			(effects
@@
 	)
 	(segment
-		(start 128.249999 119.3443)
-		(end 129.749999 119.3443)
-		(width 0.2)
-		(layer "F.Cu")
-		(net 2)
-	)
-	(segment
 		(start 143.749999 131.8443)
 		(end 148.349999 131.8443)
@@
 	)
 	(segment
+		(start 127.449999 119.3443)
+		(end 128.749999 119.3443)
+		(width 0.2)
+		(layer "F.Cu")
+		(net 2)
+	)
+	(segment
 		(start 137.709999 118.3043)
 		(end 137.949999 118.5443)
@@
 	)
 	(via
-		(at 128.449999 77.4443)
+		(at 128.749999 119.3443)
 		(size 0.6)
 		(drill 0.3)
@@
 	)
 	(via
-		(at 145.349999 107.7443)
+		(at 128.449999 77.4443)
 		(size 0.6)
 		(drill 0.3)
@@
 	)
 	(via
-		(at 148.349999 131.8443)
+		(at 145.349999 107.7443)
 		(size 0.6)
 		(drill 0.3)
@@
 	)
 	(via
-		(at 151.049999 113.6443)
+		(at 148.349999 131.8443)
 		(size 0.6)
 		(drill 0.3)
@@
 	)
 	(via
-		(at 176.849999 112.7443)
+		(at 151.049999 113.6443)
 		(size 0.6)
 		(drill 0.3)
@@
 	)
 	(via
-		(at 129.749999 119.3443)
+		(at 176.849999 112.7443)
 		(size 0.6)
 		(drill 0.3)
@@
 	)
 	(segment
-		(start 130.849999 83.262251)
-		(end 130.849999 84.2443)
-		(width 0.3)
-		(layer "F.Cu")
-		(net 4)
-	)
-	(segment
 		(start 146.449999 108.3443)
 		(end 146.449999 110.7443)
@@
 	)
 	(segment
-		(start 126.199999 121.6193)
-		(end 126.424999 121.8443)
+		(start 125.399999 119.3443)
+		(end 125.399999 120.8193)
 		(width 0.2)
 		(layer "F.Cu")
@@
 	)
 	(segment
-		(start 126.199999 119.3443)
-		(end 126.199999 121.6193)
+		(start 125.399999 120.8193)
+		(end 126.424999 121.8443)
 		(width 0.2)
 		(layer "F.Cu")
